Commit message: urdf generator completed

File: surf_rec/examples/DH_parameters/simple_2_dof.urdf (robot description, URDF)
Before this commit: robot simple_2_dof, 2 links, 1 joints
Links:
- added link base_link
- added link link_3
Joints:
- added joint joint_0: type continuous, parent base_link, child link_1, origin xyz=0  0  0 rpy=0  0  0, axis 0  0  1
- added joint joint_2: type continuous, parent link_2, child link_3, origin xyz=0.700000  0  0.000000 rpy=0.000000  0  0, axis 0  0  1
- joint joint_1: origin xyz=1.400000  0.000000  0.000000 rpy=0  0  0 -> xyz=1.400000  0  0.000000 rpy=0.000000  0  0

Commit message: urdf generator added

File: surf_rec/examples/DH_parameters/simple_2_dof.urdf (robot description, URDF)
Before this commit: robot simple_2_dof, 4 links, 3 joints
Links:
- added link link_4
Joints:
- added joint joint_3: type continuous, parent link_3, child link_4, origin xyz=0.232500  0  0.000000 rpy=0.000000  0  0, axis 0  0  1
- joint joint_0: origin xyz=0  0  0 rpy=0  0  0 -> xyz=0.000000  0  0.000000 rpy=0.000000  0  0
- joint joint_1: origin xyz=1.400000  0  0.000000 rpy=0.000000  0  0 -> xyz=0.447500  0  0.000000 rpy=1.570000  0  0
- joint joint_2: origin xyz=0.700000  0  0.000000 rpy=0.000000  0  0 -> xyz=0.330000  0  0.000000 rpy=0.000000  0  0
